File: ECE411 Preliminary Schematic/ECE411_1.kicad_pcb (KiCad board)
At the start: 2 copper layers, 14 parts, among them J2 Raspberry_Pi_4, M1 Motor_Servo, U1 XVF3800 (XM-014888-PC)

Commit message: PCB finish (maybe)
Parts:
- removed BT1: Battery, Battery:BatteryHolder_Keystone_2462_2xAA
- removed C4: 100uF, Capacitor_SMD:C_0201_0603Metric
- C1, C2, C3, C5, C6: footprint Capacitor_SMD:C_0201_0603Metric -> Capacitor_SMD:C_0603_1608Metric
- R1, R2, R3: footprint Resistor_SMD:R_0201_0603Metric -> Resistor_SMD:R_0603_1608Metric
- moved A1 93.6 mm to (155.5, 80.6)
- moved U1 63.1 mm to (84.0, 125.5)
- moved C3 58.2 mm to (148.5, 83.7), turned to -90 degrees
- moved R1 57.7 mm to (145.5, 110.0)
- moved J2 56.5 mm to (75.1, 70.9), turned to 90 degrees
- moved R2 49.7 mm to (132.7, 116.2)
- moved R3 49.7 mm to (137.7, 111.0)
- moved M1 33.3 mm to (115.5, 100.0), turned to 180 degrees
- moved C5 32.3 mm to (76.0, 111.0)
- moved C6 27.2 mm to (76.0, 106.5)
- moved C2 14.9 mm to (76.2, 88.0)
- moved C1 14.1 mm to (76.3, 82.7)
Routing:
- net +3V3: track 0.00 -> 256.8 mm
- net DIRECTION: track 0.00 -> 128.7 mm
- net PI_ESP_RX: track 0.00 -> 77.5 mm, vias 0 -> 2
- net PI_ESP_TX: track 0.00 -> 77.1 mm, vias 0 -> 1
- net AUDIO_DATA: track 0.00 -> 76.2 mm, vias 0 -> 2
- net Net-(A1-A6/IO14): track 0.00 -> 67.0 mm
- net CLK: track 0.00 -> 59.9 mm
- net Net-(M1-PWM): track 0.00 -> 25.9 mm
- net Net-(A1-TX/IO17): track 0.00 -> 23.7 mm, vias 0 -> 2
- net Net-(A1-RX/IO16): track 0.00 -> 10.7 mm
- added copper zone on B.Cu, net GND
- added copper zone on F.Cu, net GND
